Commit message: modify urdf

File: urdf/simple_car1.urdf (robot description, URDF)
Before this commit: robot simple_car, 3 links, 2 joints
Links:
- added link lidar_link, mass 0.2; collision cylinder length=0.02 radius=0.035; visual cylinder length=0.02 radius=0.035
Joints:
- added joint lidar: type fixed, parent base_link, child lidar_link, origin xyz=0.017 0.0 0.13 rpy=0 0 0

Commit message: update

File: urdf/simple_car1.urdf (robot description, URDF)
Before this commit: robot simple_car, 4 links, 3 joints
Links:
- added link back_support, mass 1.0; collision sphere radius=0.01; visual sphere radius=0.01
- added link front_support, mass 1.0; collision sphere radius=0.01; visual sphere radius=0.01
- link base_link: geometry collision box size=0.13 0.09 0.12; visual box size=0.12 0.08 0.10
Joints:
- added joint back_support: type fixed, parent base_link, child back_support, origin xyz=-0.04 0.0 0.0 rpy=0 0 0
- added joint front_support: type fixed, parent base_link, child front_support, origin xyz=0.04 0.0 0.0 rpy=0 0 0
